Commit message: Added IK model

File: Manipulator_3DoF.urdf (robot description, URDF)
Before this commit: robot spatial_3R_robot, 4 links, 3 joints
Links:
- link arm1: geometry collision box size=0.1 0.1 1.0; visual box size=0.1 0.1 1.0
- link arm2: geometry collision box size=0.1 0.1 1.0; visual box size=0.1 0.1 1.0
- link base_link: geometry collision cylinder length=0.3 radius=0.1; visual cylinder length=0.3 radius=0.1
Joints:
- joint rotation0: axis 0 0 1 -> 1 0 0; limit lower=-3.14 upper=3.14 effort=100 velocity=10 -> (none); origin xyz=0 0 0 rpy=0 0 0 -> xyz=0 0 2 rpy=0 0 0; type revolute -> continuous
- joint rotation1: axis 0 0 1 -> 0 1 0; limit lower=-3.14 upper=3.14 effort=100 velocity=10 -> (none); origin xyz=0 0 1.0 rpy=0 1.57075 0 -> xyz=0 -0.3 0 rpy=0 1.5707 0; type revolute -> continuous
- joint rotation2: axis 0 0 1 -> 0 1 0; limit lower=-3.00 upper=3.00 effort=1000 velocity=1000 -> (none); origin xyz=0 -1 0.1 rpy=0 0 0 -> xyz=0 0 -1 rpy=0 0 0; type revolute -> continuous

Commit message: Added DH solver and fixed forward kinematics model

File: Manipulator_3DoF.urdf (robot description, URDF)
Before this commit: robot spatial_3R_robot, 4 links, 3 joints
Joints:
- joint rotation1: origin xyz=0 -0.3 0 rpy=0 1.5707 0 -> xyz=0 -0.3 0 rpy=0 0 0

Commit message: Added rotation matrix to translate leg position from world coordinates to leg coordinates. Tweaked the FK model

File: Manipulator_3DoF.urdf (robot description, URDF)
Before this commit: robot spatial_3R_robot, 4 links, 3 joints
Joints:
- joint rotation1: axis 0 1 0 -> 0 -1 0; origin xyz=0 -0.3 0 rpy=0 0 0 -> xyz=0 0.3 0 rpy=0 0 0
- joint rotation2: axis 0 1 0 -> 0 -1 0

Commit message: Verified and completed the FK model

File: Manipulator_3DoF.urdf (robot description, URDF)
Before this commit: robot spatial_3R_robot, 4 links, 3 joints
Joints:
- joint rotation1: axis 0 -1 0 -> 0 1 0
- joint rotation2: axis 0 -1 0 -> 0 1 0
